Commit message: Added laser

File: src/robot/urdf/robot.xacro (robot description, xacro)
@@ -111,4 +111,25 @@
 </link>
 <!-- Link for sensors -->
+     <!-- Hokuyo Laser -->
+  <link name="hokuyo_link">
+    <collision>
+      <origin xyz="0 0 0" rpy="0 0 0"/>
+      <geometry>
+         <box size="0.1 0.1 0.1"/>
+      </geometry>
+    </collision>
+    <visual>
+      <origin xyz="0 0 0" rpy="0 0 0"/>
+      <geometry>
+	    <box size="0.1 0.1 0.1"/>
+        <!--<mesh filename="package://robot_description/meshes/hokuyo.dae"/>-->
+      </geometry>
+    </visual>
+    <inertial>
+      <mass value="1e-5" />
+      <origin xyz="0 0 0" rpy="0 0 0"/>
+      <inertia ixx="1e-6" ixy="0" ixz="0" iyy="1e-6" iyz="0" izz="1e-6" />
+    </inertial>
+  </link>
  <!--Top view rotatary Camera -->
 <!--	 <link name="camera_link_top">
@@ -123,44 +144,4 @@
 			<geometry>
 		<box size="0.04 0.024 0.003"/>
-			</geometry>
-		</visual>
-		<inertial>
-			<mass value="1e-5" />
-			<origin xyz="0 0 0" rpy="0 0 0"/>
-			<inertia ixx="1e-6" ixy="0" ixz="0" iyy="1e-6" iyz="0" izz="1e-6" />
-		</inertial>
-	</link>-->
-	<!-- Bottom view Camera -->
-	<!-- <link name="camera_link_bottom">
-		<collision name="camera_bottom_collision">
-			<origin xyz="0 0 0" rpy="0 0 0"/>
-			<geometry>
-		<box size="0.04 0.024 0.003"/>
-			</geometry>
-		</collision>
-		<visual name='camera_bottom_visual'>
-			<origin xyz="0 0 0" rpy="0 0 0"/>
-			<geometry>
-		<box size="0.04 0.024 0.003"/>
-			</geometry>
-		</visual>
-		<inertial>
-			<mass value="1e-5" />
-			<origin xyz="0 0 0" rpy="0 0 0"/>
-			<inertia ixx="1e-6" ixy="0" ixz="0" iyy="1e-6" iyz="0" izz="1e-6" />
-		</inertial>
-	</link>-->
-	<!-- Stereo Camera -->
-<!--	<link name="camera_link_stereo">
-		<collision>
-			<origin xyz="0 0 0" rpy="0 0 0"/>
-			<geometry>
-		<box size="0.085 0.024 0.03"/>
-			</geometry>
-		</collision>
-		<visual>
-			<origin xyz="0 0 0" rpy="0 0 0"/>
-			<geometry>
-		<box size="0.024 0.085 0.003"/>
 			</geometry>
 		</visual>
@@ -191,5 +172,11 @@
     <child link="caster_wheel"/>
     <origin xyz="0.24 0 0" rpy="0 0 0"/>
-</joint>
+	</joint>
+	<joint name="hokuyo_joint" type="fixed">
+    <axis xyz="0 1 0" />
+    <origin xyz="0.2 0 0.175" rpy="0 0 0"/>
+    <parent link="robot_body"/>
+    <child link="hokuyo_link"/>
+    </joint>
 <!--	<joint type="fixed" name="camera_joint_top">
 		<axis xyz="0 1 0" />
@@ -205,4 +192,7 @@
 		<material>Gazebo/Black</material>
 	</gazebo>
+	<gazebo reference="caster_wheel">
+		<material>Gazebo/Black</material>
+	</gazebo>
 	<gazebo reference="robot_body">
 		<material>Gazebo/Yellow</material>

Commit message: amcl and gmapping

File: src/robot/urdf/robot.xacro (robot description, xacro)
@@ -157,5 +157,5 @@
 		<parent link="robot_body"/>
 		<axis xyz="0 0 1" rpy="0 0 0"/>
-		<limit effort="10000" velocity="1000"/>
+		<limit effort="10000" velocity="2000"/>
 		<dynamics damping="1.0" friction="1.0"/>
 	</joint>
@@ -165,5 +165,5 @@
 		<parent link="robot_body"/>
 		<axis xyz="0 0 1" rpy="0 0 0"/>
-		<limit effort="10000" velocity="1000"/>
+		<limit effort="10000" velocity="2000"/>
 		<dynamics damping="1.0" friction="1.0"/>
 	</joint>
@@ -172,4 +172,6 @@
     <child link="caster_wheel"/>
     <origin xyz="0.24 0 0" rpy="0 0 0"/>
+	<limit effort="10000" velocity="2000"/>
+	<dynamics damping="1.0" friction="1.0"/>
 	</joint>
 	<joint name="hokuyo_joint" type="fixed">

Commit message: amcl and move_base added

File: src/robot/urdf/robot.xacro (robot description, xacro)
@@ -8,5 +8,4 @@
 	<joint name="robot_footprint_joint" type="fixed">
 		<origin xyz="-0.1 0 0" rpy="0 0 0" />
-<!-- x poits towards back of body, y upwards -->
 		<parent link="robot_footprint"/>
 		<child link="robot_body" />
@@ -161,5 +160,5 @@
 	</joint>
 	<joint type="continuous" name="right_wheel_hinge">
-		<origin xyz="0.05 -0.175 0" rpy="${pi/2} 0 0"/>
+		<origin xyz="0.05 -0.175 0" rpy="-${pi/2} 0  0 "/>
 		<child link="right_wheel"/>
 		<parent link="robot_body"/>
